File: EtherCAT_shield_v1.sch (KiCad schematic (older format))
At the start: 58 parts, among them J1 RJ45-PULSETRANS, J2 RJ45-PULSETRANS, J3 GS3, J4 GS3, J5 GS3, J6 GS3, J7 GS2, J8 GS2, P1 CONN_02X10, P2 CONN_02X19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

Commit message: CHS GNDとPCB GNDを抵抗で接続
Parts:
- added R40, R41: R, Resistors_SMD:R_1210, symbol R
Connections:
- net GND: now also R40.2, R41.2
- net GNDPWR: now also R40.1, R41.1
Changed lines of the file:
@@
 Wire Wire Line
 	8800 5650 8800 4700
+$Comp
+L GNDPWR #PWR046
+U 1 1 58E26654
+P 10400 6000
+F 0 "#PWR046" H 10400 5800 50  0001 C CNN
+F 1 "GNDPWR" H 10400 5870 50  0000 C CNN
+F 2 "" H 10400 5950 50  0001 C CNN
+F 3 "" H 10400 5950 50  0001 C CNN
+	1    10400 6000
+	1    0    0    -1
+$EndComp
+$Comp
+L GND #PWR047
+U 1 1 58E271DD
+P 10000 6000
+F 0 "#PWR047" H 10000 5750 50  0001 C CNN
+F 1 "GND" H 10000 5850 50  0000 C CNN
+F 2 "" H 10000 6000 50  0000 C CNN
+F 3 "" H 10000 6000 50  0000 C CNN
+	1    10000 6000
+	1    0    0    -1
+$EndComp
+$Comp
+L GNDPWR #PWR048
+U 1 1 58E28308
+P 10400 4300
+F 0 "#PWR048" H 10400 4100 50  0001 C CNN
+F 1 "GNDPWR" H 10400 4170 50  0000 C CNN
+F 2 "" H 10400 4250 50  0001 C CNN
+F 3 "" H 10400 4250 50  0001 C CNN
+	1    10400 4300
+	1    0    0    -1
+$EndComp
+$Comp
+L GND #PWR049
+U 1 1 58E2841B
+P 10000 4300
+F 0 "#PWR049" H 10000 4050 50  0001 C CNN
+F 1 "GND" H 10000 4150 50  0000 C CNN
+F 2 "" H 10000 4300 50  0000 C CNN
+F 3 "" H 10000 4300 50  0000 C CNN
+	1    10000 4300
+	1    0    0    -1
+$EndComp
+$Comp
+L R R40
+U 1 1 58E284F6
+P 10200 4250
+F 0 "R40" V 10280 4250 50  0000 C CNN
+F 1 "R" V 10200 4250 50  0000 C CNN
+F 2 "Resistors_SMD:R_1210" V 10130 4250 50  0001 C CNN
+F 3 "" H 10200 4250 50  0001 C CNN
+	1    10200 4250
+	0    1    1    0
+$EndComp
+$Comp
+L R R41
+U 1 1 58E28CC4
+P 10200 5950
+F 0 "R41" V 10280 5950 50  0000 C CNN
+F 1 "R" V 10200 5950 50  0000 C CNN
+F 2 "Resistors_SMD:R_1210" V 10130 5950 50  0001 C CNN
+F 3 "" H 10200 5950 50  0001 C CNN
+	1    10200 5950
+	0    1    1    0
+$EndComp
+Wire Wire Line
+	10350 5950 10400 5950
+Wire Wire Line
+	10400 5950 10400 6000
+Wire Wire Line
+	10000 6000 10000 5950
+Wire Wire Line
+	10000 5950 10050 5950
+Wire Wire Line
+	10350 4250 10400 4250
+Wire Wire Line
+	10400 4250 10400 4300
+Wire Wire Line
+	10050 4250 10000 4250
+Wire Wire Line
+	10000 4250 10000 4300
 $EndSCHEMATC

Commit message: 抵抗とかコンデンサを追加
Parts:
- added C30, C31: 10u, Capacitors_SMD:C_0805, symbol C
Connections:
- net +3V3: now also C31.1
- net +5V: now also C30.1
- net GND: now also C30.2, C31.2
Changed lines of the file:
@@
 Wire Wire Line
 	10000 4250 10000 4300
+$Comp
+L +3V3 #PWR050
+U 1 1 58E4EAB7
+P 1850 700
+F 0 "#PWR050" H 1850 550 50  0001 C CNN
+F 1 "+3V3" H 1850 840 50  0000 C CNN
+F 2 "" H 1850 700 50  0000 C CNN
+F 3 "" H 1850 700 50  0000 C CNN
+	1    1850 700
+	1    0    0    -1
+$EndComp
+$Comp
+L +5V #PWR051
+U 1 1 58E4ED74
+P 1550 700
+F 0 "#PWR051" H 1550 550 50  0001 C CNN
+F 1 "+5V" H 1550 840 50  0000 C CNN
+F 2 "" H 1550 700 50  0000 C CNN
+F 3 "" H 1550 700 50  0000 C CNN
+	1    1550 700
+	1    0    0    -1
+$EndComp
+$Comp
+L C C31
+U 1 1 58E4F47A
+P 1850 850
+F 0 "C31" H 1875 950 50  0000 L CNN
+F 1 "10u" H 1875 750 50  0000 L CNN
+F 2 "Capacitors_SMD:C_0805" H 1888 700 50  0001 C CNN
+F 3 "" H 1850 850 50  0001 C CNN
+	1    1850 850
+	1    0    0    -1
+$EndComp
+$Comp
+L C C30
+U 1 1 58E4F5C4
+P 1550 850
+F 0 "C30" H 1575 950 50  0000 L CNN
+F 1 "10u" H 1575 750 50  0000 L CNN
+F 2 "Capacitors_SMD:C_0805" H 1588 700 50  0001 C CNN
+F 3 "" H 1550 850 50  0001 C CNN
+	1    1550 850
+	1    0    0    -1
+$EndComp
+$Comp
+L GND #PWR052
+U 1 1 58E4F6F0
+P 1550 1000
+F 0 "#PWR052" H 1550 750 50  0001 C CNN
+F 1 "GND" H 1550 850 50  0000 C CNN
+F 2 "" H 1550 1000 50  0000 C CNN
+F 3 "" H 1550 1000 50  0000 C CNN
+	1    1550 1000
+	1    0    0    -1
+$EndComp
+$Comp
+L GND #PWR053
+U 1 1 58E4F80F
+P 1850 1000
+F 0 "#PWR053" H 1850 750 50  0001 C CNN
+F 1 "GND" H 1850 850 50  0000 C CNN
+F 2 "" H 1850 1000 50  0000 C CNN
+F 3 "" H 1850 1000 50  0000 C CNN
+	1    1850 1000
+	1    0    0    -1
+$EndComp
 $EndSCHEMATC

Commit message: 値ふってBOM作成
Parts:
- R3: value 0R -> 0
Connections:
- no-connect marks 9 -> 53
Changed lines of the file:
@@
 LIBS:valves
 LIBS:mylib
+LIBS:analog_devices
 LIBS:EtherCAT_shield_v1-cache
 EELAYER 25 0
@@
 P 7750 2950
 F 0 "R3" V 7830 2950 50  0000 C CNN
-F 1 "0R" V 7750 2950 50  0000 C CNN
+F 1 "0" V 7750 2950 50  0000 C CNN
 F 2 "Resistors_SMD:R_0603" V 7680 2950 50  0001 C CNN
 F 3 "" H 7750 2950 50  0000 C CNN
@@
 Text GLabel 1700 5700 0    60   Input ~ 0
 PC10
-Text GLabel 3550 6050 2    60   Input ~ 0
-PA6
 Text GLabel 3450 6400 0    60   Input ~ 0
 PA7
@@
 	1    0    0    -1
 $EndComp
+NoConn ~ 1750 5800
+NoConn ~ 1750 5900
+NoConn ~ 1750 6000
+NoConn ~ 1750 6300
+NoConn ~ 1750 6400
+NoConn ~ 1750 6500
+NoConn ~ 1750 7100
+NoConn ~ 1750 7200
+NoConn ~ 1750 7300
+NoConn ~ 1750 7400
+NoConn ~ 1750 7500
+NoConn ~ 2250 7500
+NoConn ~ 2250 7400
+NoConn ~ 2250 7200
+NoConn ~ 2250 7100
+NoConn ~ 2250 7000
+NoConn ~ 2250 6800
+NoConn ~ 2250 5900
+NoConn ~ 2250 5800
+NoConn ~ 2250 5700
+NoConn ~ 4150 5800
+NoConn ~ 4150 5900
+NoConn ~ 4150 6000
+NoConn ~ 4150 6200
+NoConn ~ 4150 6600
+NoConn ~ 4150 6700
+NoConn ~ 4150 6800
+NoConn ~ 4150 7000
+NoConn ~ 4150 7100
+NoConn ~ 4150 7200
+NoConn ~ 4150 7300
+NoConn ~ 4150 7400
+NoConn ~ 4150 7500
+NoConn ~ 4650 7300
+NoConn ~ 4650 7100
+NoConn ~ 4650 7000
+NoConn ~ 4650 6900
+NoConn ~ 4650 6400
+NoConn ~ 4650 6300
+NoConn ~ 4650 6200
+NoConn ~ 4650 6000
+NoConn ~ 4650 5900
+NoConn ~ 4650 5800
+NoConn ~ 4650 5700
+Text GLabel 3550 6050 2    60   Input ~ 0
+PA6
 $EndSCHEMATC
